File: ematch-driver.sch (KiCad schematic (older format))
At the start: 7 parts, among them Q2 Q_NMOS_GSD, Q3 Q_PMOS_GDS

Commit message: fucking mac windows manager is a pile of shit
Parts:
- added D?: TVS, do-214ac, symbol TVS
Changed lines of the file:
@@
 Connection ~ 3050 2900
 Wire Wire Line
-	4100 5300 4100 5750
+	4050 6350 4050 6800
 Wire Wire Line
 	3550 4100 3550 4900
@@
 Text HLabel 4100 5000 2    60   Input ~ 0
 EMATCH_VCC
-Text HLabel 4100 5300 2    60   Input ~ 0
+Text HLabel 4050 6350 2    60   Input ~ 0
 EMATCH_GND
 Text HLabel 3050 3000 3    60   Input ~ 0
@@
 Text HLabel 3550 5500 3    60   Input ~ 0
 GND
-Text HLabel 4100 5750 3    60   Input ~ 0
+Text HLabel 4050 6800 3    60   Input ~ 0
 GND
 Wire Wire Line
@@
 	1    0    0    1
 $EndComp
+$Comp
+L TVS D?
+U 1 1 58A0E744
+P 5200 5300
+F 0 "D?" H 5200 5450 50  0000 C CNN
+F 1 "TVS" H 5200 5150 50  0000 C CNN
+F 2 "do-214ac" H 5550 4550 50  0000 C CNN
+F 3 "" H 5200 5300 50  0000 C CNN
+	1    5200 5300
+	1    0    0    -1
+$EndComp
 $EndSCHEMATC

Commit message: Updates from 2018 rev
Parts:
- D17: renamed from D?; footprint do-214ac -> Diodes_SMD:D_SMA_Handsoldering; digikey part no (none) -> SMAJ30CALFTR-ND
- Q2: footprint TO_SOT_Packages_SMD:SOT-23 -> TO_SOT_Packages_SMD:SOT-23_Handsoldering
- Q3: digikey part no (none) -> NTD2955T4GOSCT-ND; digikey part number NTD2955T4GOSCT-ND -> (none)
- R9: digikey part no PLT0603-500ATR-ND -> 311-499HRCT-ND
Connections:
- net EMATCH_GND: now also D17.2
- net EMATCH_VCC: now also D17.1
Other:
- moved on the sheet: D20
Changed lines of the file:
@@
 $Descr A4 11693 8268
 encoding utf-8
-Sheet 2 9
+Sheet 3 9
 Title ""
 Date ""
@@
 AR Path="/56EAA68A/56CFCF8E" Ref="R27"  Part="1"
 AR Path="/56EAA6CF/56CFCF8E" Ref="R30"  Part="1"
-F 0 "R9" V 3080 4100 50  0000 C CNN
+F 0 "R18" V 3080 4100 50  0000 C CNN
 F 1 "500" V 3000 4100 50  0000 C CNN
 F 2 "Resistors_SMD:R_0603_HandSoldering" V 2930 4100 50  0001 C CNN
 F 3 "" H 3000 4100 50  0000 C CNN
-F 4 "PLT0603-500ATR-ND" V 3000 4100 60  0001 C CNN "digikey part no"
+F 4 "311-499HRCT-ND" V 3000 4100 60  0001 C CNN "digikey part no"
 	1    3000 4100
 	0    1    1    0
@@
 AR Path="/56EAA68A/56CFD0B3" Ref="R28"  Part="1"
 AR Path="/56EAA6CF/56CFD0B3" Ref="R31"  Part="1"
-F 0 "R10" V 3130 2600 50  0000 C CNN
+F 0 "R19" V 3130 2600 50  0000 C CNN
 F 1 "10k" V 3050 2600 50  0000 C CNN
 F 2 "Resistors_SMD:R_0603_HandSoldering" V 2980 2600 50  0001 C CNN
@@
 AR Path="/56EAA68A/56CFDBA4" Ref="Q14"  Part="1"
 AR Path="/56EAA6CF/56CFDBA4" Ref="Q16"  Part="1"
-F 0 "Q2" H 3750 2150 50  0000 R CNN
+F 0 "Q8" H 3750 2150 50  0000 R CNN
 F 1 "Q_NMOS_GSD" H 4100 2050 50  0000 R CNN
-F 2 "TO_SOT_Packages_SMD:SOT-23" H 3650 2200 50  0001 C CNN
+F 2 "TO_SOT_Packages_SMD:SOT-23_Handsoldering" H 3650 2200 50  0001 C CNN
 F 3 "http://toshiba.semicon-storage.com/info/docget.jsp?did=13879&prodName=SSM3K324R" H 3450 2100 50  0001 C CNN
 F 4 "SSM3K324RLFCT-ND" H 3450 2100 60  0001 C CNN "digikey part no"
@@
 AR Path="/56EAA68A/56CFDBE5" Ref="R29"  Part="1"
 AR Path="/56EAA6CF/56CFDBE5" Ref="R32"  Part="1"
-F 0 "R11" V 3630 1400 50  0000 C CNN
+F 0 "R20" V 3630 1400 50  0000 C CNN
 F 1 "10k" V 3550 1400 50  0000 C CNN
 F 2 "Resistors_SMD:R_0603_HandSoldering" V 3480 1400 50  0001 C CNN
@@
 AR Path="/56EAA68A/56CFDC9F" Ref="D14"  Part="1"
 AR Path="/56EAA6CF/56CFDC9F" Ref="D16"  Part="1"
-F 0 "D2" H 3900 4750 50  0000 C CNN
+F 0 "D8" H 3900 4750 50  0000 C CNN
 F 1 "D" H 3900 4550 50  0000 C CNN
 F 2 "Diodes_SMD:SOD-123" H 3900 4650 50  0001 C CNN
@@
 AR Path="/56EAA68A/56CFDD3A" Ref="D13"  Part="1"
 AR Path="/56EAA6CF/56CFDD3A" Ref="D15"  Part="1"
-F 0 "D1" H 3550 5200 50  0000 C CNN
+F 0 "D7" H 3550 5200 50  0000 C CNN
 F 1 "ZENER" H 3550 5000 50  0000 C CNN
 F 2 "Diodes_SMD:SOD-123" H 3550 5100 50  0001 C CNN
@@
 Connection ~ 3050 2900
 Wire Wire Line
-	4050 6350 4050 6800
+	4100 5600 4100 6050
 Wire Wire Line
 	3550 4100 3550 4900
@@
 Text HLabel 4100 5000 2    60   Input ~ 0
 EMATCH_VCC
-Text HLabel 4050 6350 2    60   Input ~ 0
+Text HLabel 4100 5600 2    60   Input ~ 0
 EMATCH_GND
 Text HLabel 3050 3000 3    60   Input ~ 0
@@
 Text HLabel 3550 5500 3    60   Input ~ 0
 GND
-Text HLabel 4050 6800 3    60   Input ~ 0
+Text HLabel 4100 6050 3    60   Input ~ 0
 GND
 Wire Wire Line
@@
 AR Path="/56EAA681/5743D9FD" Ref="Q13"  Part="1"
 AR Path="/56EAA6CF/5743D9FD" Ref="Q17"  Part="1"
-F 0 "Q3" H 4300 1800 50  0000 R CNN
+F 0 "Q9" H 4300 1800 50  0000 R CNN
 F 1 "Q_PMOS_GDS" H 4650 1700 50  0000 R CNN
 F 2 "TO_SOT_Packages_SMD:TO-252-2Lead" H 4200 1850 50  0001 C CNN
 F 3 "https://www.onsemi.com/pub_link/Collateral/NTD2955-D.PDF" H 4000 1750 50  0001 C CNN
-F 4 "NTD2955T4GOSCT-ND	" H 4000 1750 60  0001 C CNN "digikey part number"
+F 4 "NTD2955T4GOSCT-ND	" H 4000 1750 60  0001 C CNN "digikey part no"
 	1    4000 1750
 	1    0    0    1
 $EndComp
 $Comp
-L TVS D?
+L TVS D17
 U 1 1 58A0E744
-P 5200 5300
-F 0 "D?" H 5200 5450 50  0000 C CNN
-F 1 "TVS" H 5200 5150 50  0000 C CNN
-F 2 "do-214ac" H 5550 4550 50  0000 C CNN
-F 3 "" H 5200 5300 50  0000 C CNN
-	1    5200 5300
-	1    0    0    -1
+P 4100 5300
+AR Path="/56CFDAEF/58A0E744" Ref="D17"  Part="1"
+AR Path="/56EAA678/58A0E744" Ref="D21"  Part="1"
+AR Path="/56D0EADF/58A0E744" Ref="D18"  Part="1"
+AR Path="/56D11458/58A0E744" Ref="D19"  Part="1"
+AR Path="/56EA4F7F/58A0E744" Ref="D20"  Part="1"
+AR Path="/56EAA681/58A0E744" Ref="D22"  Part="1"
+AR Path="/56EAA68A/58A0E744" Ref="D23"  Part="1"
+AR Path="/56EAA6CF/58A0E744" Ref="D24"  Part="1"
+F 0 "D20" H 4100 5450 50  0000 C CNN
+F 1 "TVS" H 4100 5150 50  0000 C CNN
+F 2 "Diodes_SMD:D_SMA_Handsoldering" H 4150 5500 50  0001 C CNN
+F 3 "" H 4100 5300 50  0000 C CNN
+F 4 "SMAJ30CALFTR-ND" H 4100 5300 60  0001 C CNN "digikey part no"
+	1    4100 5300
+	0    1    1    0
 $EndComp
 $EndSCHEMATC
