File: remote-pallet.kicad_pcb (KiCad board)
At the start: 2 copper layers, 90 x 90 mm, 87 parts, among them J1 Power, M0 E-MATCH, M1 E-MATCH, M2 E-MATCH, M3 E-MATCH, M4 E-MATCH, M5 E-MATCH, M6 E-MATCH, M7 E-MATCH, Q1 EMatch Test, Q10 Q_NMOS_GSD, Q11 Q_PMOS_GDS, Q12 Q_NMOS_GSD, Q13 Q_PMOS_GDS, Q14 Q_NMOS_GSD, Q15 Q_PMOS_GDS, Q16 Q_NMOS_GSD, Q17 Q_PMOS_GDS, Q2 Q_NMOS_GSD, Q3 Q_PMOS_GDS, Q4 Q_NMOS_GSD, Q5 Q_PMOS_GDS, Q6 Q_NMOS_GSD, Q7 Q_PMOS_GDS, Q8 Q_NMOS_GSD, Q9 Q_PMOS_GDS, SW1 Power, SW2 Arm Hardware, U1 Photon Power, U2 PHOTON, U3 Armed Sense

Commit message: Updates from 2018 rev
Parts:
- added D17: TVS, Diodes_SMD:D_SMA_Handsoldering, B.Cu at (170.1, 122.2)
- added D18: TVS, Diodes_SMD:D_SMA_Handsoldering, B.Cu at (170.2, 103.3)
- added D19: TVS, Diodes_SMD:D_SMA_Handsoldering, B.Cu at (170.0, 84.8)
- added D20: TVS, Diodes_SMD:D_SMA_Handsoldering, B.Cu at (169.9, 67.6)
- added D21: TVS, Diodes_SMD:D_SMA_Handsoldering, B.Cu at (103.3, 122.5)
- added D22: TVS, Diodes_SMD:D_SMA_Handsoldering, B.Cu at (103.3, 103.6)
- added D23: TVS, Diodes_SMD:D_SMA_Handsoldering, B.Cu at (103.4, 85.0)
- added D24: TVS, Diodes_SMD:D_SMA_Handsoldering, B.Cu at (103.4, 67.4)
- M0, M1, M2, M3, M4, M5, M6, M7: footprint Terminal_Blocks:TerminalBlock_Pheonix_PT-3.5mm_2pol -> Terminal_Blocks:TerminalBlock_Altech_AK300-2_P5.00mm
- Q1, Q10, Q12, Q14, Q16, Q2, Q4, Q6, Q8: footprint TO_SOT_Packages_SMD:SOT-23 -> TO_SOT_Packages_SMD:SOT-23_Handsoldering
- moved G*** 72.8 mm to (151.1, 131.9), turned to 180 degrees
- moved Q3 8.71 mm to (164.5, 112.5), turned to 180 degrees
- moved Q5 6.48 mm to (164.5, 98.8), turned to 180 degrees
- moved Q17 6.48 mm to (109.5, 63.4), turned to 0 degrees
- moved Q15 5.16 mm to (109.5, 80.8), turned to 0 degrees
- moved Q7 5.13 mm to (164.4, 84.2), turned to 180 degrees
- moved Q9 5.06 mm to (164.5, 68.4), turned to 180 degrees
- moved M7 4.84 mm to (99.1, 65.0)
- moved M0 4.16 mm to (174.9, 124.8)
- moved M6 3.58 mm to (99.2, 82.5)
- moved M3 3.36 mm to (174.9, 70.1)
- moved M4 2.94 mm to (99.1, 120.0)
- moved Q13 2.84 mm to (109.6, 99.4), turned to 0 degrees
- moved M2 2.27 mm to (174.9, 87.5)
- moved Q11 2.02 mm to (109.5, 118.3), turned to 0 degrees
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Routing:
- net /ematch-7/EMATCH_VCC: track 79.5 -> 97.7 mm, vias 1 -> 0
- net /ematch-6/EMATCH_VCC: track 68.7 -> 85.5 mm, vias 1 -> 0
- net /ematch-5/EMATCH_VCC: track 57.3 -> 71.2 mm, vias 1 -> 0
- net /ematch-1/EMATCH_VCC: track 58.8 -> 71.4 mm
- net /ematch-3/EMATCH_VCC: track 101.9 -> 114.3 mm
- net /ematch-0/EMATCH_VCC: track 37.8 -> 50.0 mm
- net /ematch-4/EMATCH_VCC: track 45.7 -> 55.1 mm, vias 1 -> 0
- net Net-(Q14-Pad3): track 71.8 -> 80.9 mm
- net /ematch-2/EMATCH_VCC: track 79.9 -> 87.2 mm
- net Net-(Q12-Pad3): track 77.6 -> 84.3 mm
- net Armed: track 71.7 -> 75.9 mm
- net Net-(Q10-Pad3): track 97.8 -> 101.5 mm
- net Fire0: track 14.7 -> 18.0 mm
- net Net-(Q2-Pad3): track 61.2 -> 58.0 mm
- net Fire3: track 20.1 -> 23.2 mm
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Other:
- net class Default: clearance 0.2 -> 0.26; trace_width 0.25 -> 0.26
- rule trace_clearance: 0.2 -> 0.26
- board text added: "M0"
- board text added: "M1"
- board text added: "M2"
- board text added: "M3"
- board text added: "M4"
- board text added: "M5"
- board text added: "M6"
- board text added: "M7"
