File: remote-pallet.sch (KiCad schematic (older format))
At the start: 26 parts, among them J1 Power, M0 E-MATCH, M1 E-MATCH, M2 E-MATCH, M3 E-MATCH, M4 E-MATCH, M5 E-MATCH, M6 E-MATCH, M7 E-MATCH, Q1 EMatch Test, SW1 Power, SW2 Arm Hardware, U1 Photon Power, U2 PHOTON, U3 Armed Sense

Commit message: Updates from 2018 rev
Parts:
- M0, M1, M2, M3, M4, M5, M6, M7: footprint Terminal_Blocks:TerminalBlock_Pheonix_PT-3.5mm_2pol -> Terminal_Blocks:TerminalBlock_Altech_AK300-2_P5.00mm; digikey part no ED2740-ND -> 277-2518-ND
- Q1: footprint TO_SOT_Packages_SMD:SOT-23 -> TO_SOT_Packages_SMD:SOT-23_Handsoldering; digikey part no BSS84PH6433XTMA1CT-ND -> SSM3K324RLFCT-ND
Changed lines of the file:
@@
 $EndComp
 $Comp
-L GND #PWR4
+L GND #PWR01
 U 1 1 56CFD8F0
 P 2350 1400
-F 0 "#PWR4" H 2350 1150 50  0001 C CNN
+F 0 "#PWR01" H 2350 1150 50  0001 C CNN
 F 1 "GND" H 2350 1250 50  0000 C CNN
 F 2 "" H 2350 1400 50  0000 C CNN
@@
 $EndSheet
 $Comp
-L GND #PWR6
+L GND #PWR02
 U 1 1 56D28AC8
 P 5050 2800
-F 0 "#PWR6" H 5050 2550 50  0001 C CNN
+F 0 "#PWR02" H 5050 2550 50  0001 C CNN
 F 1 "GND" H 5050 2650 50  0000 C CNN
 F 2 "" H 5050 2800 50  0000 C CNN
@@
 $EndComp
 $Comp
-L GND #PWR7
+L GND #PWR03
 U 1 1 56D28F92
 P 5050 3800
-F 0 "#PWR7" H 5050 3550 50  0001 C CNN
+F 0 "#PWR03" H 5050 3550 50  0001 C CNN
 F 1 "GND" H 5050 3650 50  0000 C CNN
 F 2 "" H 5050 3800 50  0000 C CNN
@@
 $EndComp
 $Comp
-L GND #PWR8
+L GND #PWR04
 U 1 1 56D2B57F
 P 5050 4750
-F 0 "#PWR8" H 5050 4500 50  0001 C CNN
+F 0 "#PWR04" H 5050 4500 50  0001 C CNN
 F 1 "GND" H 5050 4600 50  0000 C CNN
 F 2 "" H 5050 4750 50  0000 C CNN
@@
 $EndSheet
 $Comp
-L GND #PWR9
+L GND #PWR05
 U 1 1 56EA4F8F
 P 5050 5750
-F 0 "#PWR9" H 5050 5500 50  0001 C CNN
+F 0 "#PWR05" H 5050 5500 50  0001 C CNN
 F 1 "GND" H 5050 5600 50  0000 C CNN
 F 2 "" H 5050 5750 50  0000 C CNN
@@
 $EndSheet
 $Comp
-L GND #PWR15
+L GND #PWR06
 U 1 1 56EAA6B2
 P 8050 2800
-F 0 "#PWR15" H 8050 2550 50  0001 C CNN
+F 0 "#PWR06" H 8050 2550 50  0001 C CNN
 F 1 "GND" H 8050 2650 50  0000 C CNN
 F 2 "" H 8050 2800 50  0000 C CNN
@@
 $EndComp
 $Comp
-L GND #PWR16
+L GND #PWR07
 U 1 1 56EAA6B8
 P 8050 3800
-F 0 "#PWR16" H 8050 3550 50  0001 C CNN
+F 0 "#PWR07" H 8050 3550 50  0001 C CNN
 F 1 "GND" H 8050 3650 50  0000 C CNN
 F 2 "" H 8050 3800 50  0000 C CNN
@@
 $EndComp
 $Comp
-L GND #PWR17
+L GND #PWR08
 U 1 1 56EAA6C2
 P 8050 4750
-F 0 "#PWR17" H 8050 4500 50  0001 C CNN
+F 0 "#PWR08" H 8050 4500 50  0001 C CNN
 F 1 "GND" H 8050 4600 50  0000 C CNN
 F 2 "" H 8050 4750 50  0000 C CNN
@@
 $EndSheet
 $Comp
-L GND #PWR18
+L GND #PWR09
 U 1 1 56EAA6DF
 P 8050 5750
-F 0 "#PWR18" H 8050 5500 50  0001 C CNN
+F 0 "#PWR09" H 8050 5500 50  0001 C CNN
 F 1 "GND" H 8050 5600 50  0000 C CNN
 F 2 "" H 8050 5750 50  0000 C CNN
@@
 $EndComp
 $Comp
-L GND #PWR2
+L GND #PWR010
 U 1 1 56EC9075
 P 900 3050
-F 0 "#PWR2" H 900 2800 50  0001 C CNN
+F 0 "#PWR010" H 900 2800 50  0001 C CNN
 F 1 "GND" H 900 2900 50  0000 C CNN
 F 2 "" H 900 3050 50  0000 C CNN
@@
 $EndComp
 $Comp
-L GND #PWR22
+L GND #PWR011
 U 1 1 56ED2DA7
 P 10050 5950
-F 0 "#PWR22" H 10050 5700 50  0001 C CNN
+F 0 "#PWR011" H 10050 5700 50  0001 C CNN
 F 1 "GND" H 10050 5800 50  0000 C CNN
 F 2 "" H 10050 5950 50  0000 C CNN
@@
 $EndComp
 $Comp
-L GND #PWR21
+L GND #PWR012
 U 1 1 56ED2FF7
 P 10050 4850
-F 0 "#PWR21" H 10050 4600 50  0001 C CNN
+F 0 "#PWR012" H 10050 4600 50  0001 C CNN
 F 1 "GND" H 10050 4700 50  0000 C CNN
 F 2 "" H 10050 4850 50  0000 C CNN
@@
 $EndComp
 $Comp
-L GND #PWR20
+L GND #PWR013
 U 1 1 56ED317C
 P 10050 3850
-F 0 "#PWR20" H 10050 3600 50  0001 C CNN
+F 0 "#PWR013" H 10050 3600 50  0001 C CNN
 F 1 "GND" H 10050 3700 50  0000 C CNN
 F 2 "" H 10050 3850 50  0000 C CNN
@@
 $EndComp
 $Comp
-L GND #PWR19
+L GND #PWR014
 U 1 1 56ED3301
 P 10050 2850
-F 0 "#PWR19" H 10050 2600 50  0001 C CNN
+F 0 "#PWR014" H 10050 2600 50  0001 C CNN
 F 1 "GND" H 10050 2700 50  0000 C CNN
 F 2 "" H 10050 2850 50  0000 C CNN
@@
 $EndComp
 $Comp
-L GND #PWR11
+L GND #PWR015
 U 1 1 56ED3D0E
 P 7050 2850
-F 0 "#PWR11" H 7050 2600 50  0001 C CNN
+F 0 "#PWR015" H 7050 2600 50  0001 C CNN
 F 1 "GND" H 7050 2700 50  0000 C CNN
 F 2 "" H 7050 2850 50  0000 C CNN
@@
 $EndComp
 $Comp
-L GND #PWR12
+L GND #PWR016
 U 1 1 56ED3E93
 P 7050 3850
-F 0 "#PWR12" H 7050 3600 50  0001 C CNN
+F 0 "#PWR016" H 7050 3600 50  0001 C CNN
 F 1 "GND" H 7050 3700 50  0000 C CNN
 F 2 "" H 7050 3850 50  0000 C CNN
@@
 $EndComp
 $Comp
-L GND #PWR13
+L GND #PWR017
 U 1 1 56ED4034
 P 7050 4850
-F 0 "#PWR13" H 7050 4600 50  0001 C CNN
+F 0 "#PWR017" H 7050 4600 50  0001 C CNN
 F 1 "GND" H 7050 4700 50  0000 C CNN
 F 2 "" H 7050 4850 50  0000 C CNN
@@
 $EndComp
 $Comp
-L GND #PWR14
+L GND #PWR018
 U 1 1 56ED41B9
 P 7050 5800
-F 0 "#PWR14" H 7050 5550 50  0001 C CNN
+F 0 "#PWR018" H 7050 5550 50  0001 C CNN
 F 1 "GND" H 7050 5650 50  0000 C CNN
 F 2 "" H 7050 5800 50  0000 C CNN
@@
 F 0 "Q1" H 4650 1300 50  0000 R CNN
 F 1 "EMatch Test" H 5000 1200 50  0000 R CNN
-F 2 "TO_SOT_Packages_SMD:SOT-23" H 4550 1350 50  0001 C CNN
+F 2 "TO_SOT_Packages_SMD:SOT-23_Handsoldering" H 4550 1350 50  0001 C CNN
 F 3 "" H 4350 1250 50  0000 C CNN
-F 4 "BSS84PH6433XTMA1CT-ND" H 4350 1250 60  0001 C CNN "digikey part no"
+F 4 "SSM3K324RLFCT-ND" H 4350 1250 60  0001 C CNN "digikey part no"
 	1    4350 1250
 	1    0    0    -1
@@
 3.3V
 $Comp
-L GND #PWR10
+L GND #PWR019
 U 1 1 56EB2D78
 P 6250 1350
-F 0 "#PWR10" H 6250 1100 50  0001 C CNN
+F 0 "#PWR019" H 6250 1100 50  0001 C CNN
 F 1 "GND" H 6250 1200 50  0000 C CNN
 F 2 "" H 6250 1350 50  0000 C CNN
@@
 F 0 "M0" H 7050 2560 50  0000 C CNN
 F 1 "E-MATCH" H 7050 2430 50  0000 C CNN
-F 2 "Terminal_Blocks:TerminalBlock_Pheonix_PT-3.5mm_2pol" H 7050 2500 50  0001 C CNN
+F 2 "Terminal_Blocks:TerminalBlock_Altech_AK300-2_P5.00mm" H 7050 2500 50  0001 C CNN
 F 3 "" H 7050 2500 50  0000 C CNN
-F 4 "ED2740-ND" H 7050 2500 60  0001 C CNN "digikey part no"
+F 4 "277-2518-ND" H 7050 2500 60  0001 C CNN "digikey part no"
 	1    7050 2500
 	0    1    1    0
@@
 F 0 "M1" H 7050 3610 50  0000 C CNN
 F 1 "E-MATCH" H 7050 3480 50  0000 C CNN
-F 2 "Terminal_Blocks:TerminalBlock_Pheonix_PT-3.5mm_2pol" H 7050 3550 50  0001 C CNN
+F 2 "Terminal_Blocks:TerminalBlock_Altech_AK300-2_P5.00mm" H 7050 3550 50  0001 C CNN
 F 3 "" H 7050 3550 50  0000 C CNN
-F 4 "ED2740-ND" H 7050 3550 60  0001 C CNN "digikey part no"
+F 4 "277-2518-ND" H 7050 3550 60  0001 C CNN "digikey part no"
 	1    7050 3550
 	0    1    1    0
@@
 F 0 "M2" H 7050 4510 50  0000 C CNN
 F 1 "E-MATCH" H 7050 4380 50  0000 C CNN
-F 2 "Terminal_Blocks:TerminalBlock_Pheonix_PT-3.5mm_2pol" H 7050 4450 50  0001 C CNN
+F 2 "Terminal_Blocks:TerminalBlock_Altech_AK300-2_P5.00mm" H 7050 4450 50  0001 C CNN
 F 3 "" H 7050 4450 50  0000 C CNN
-F 4 "ED2740-ND" H 7050 4450 60  0001 C CNN "digikey part no"
+F 4 "277-2518-ND" H 7050 4450 60  0001 C CNN "digikey part no"
 	1    7050 4450
 	0    1    1    0
@@
 F 0 "M3" H 7050 5510 50  0000 C CNN
 F 1 "E-MATCH" H 7050 5380 50  0000 C CNN
-F 2 "Terminal_Blocks:TerminalBlock_Pheonix_PT-3.5mm_2pol" H 7050 5450 50  0001 C CNN
+F 2 "Terminal_Blocks:TerminalBlock_Altech_AK300-2_P5.00mm" H 7050 5450 50  0001 C CNN
 F 3 "" H 7050 5450 50  0000 C CNN
-F 4 "ED2740-ND" H 7050 5450 60  0001 C CNN "digikey part no"
+F 4 "277-2518-ND" H 7050 5450 60  0001 C CNN "digikey part no"
 	1    7050 5450
 	0    1    1    0
@@
 F 0 "M4" H 10050 2560 50  0000 C CNN
 F 1 "E-MATCH" H 10050 2430 50  0000 C CNN
-F 2 "Terminal_Blocks:TerminalBlock_Pheonix_PT-3.5mm_2pol" H 10050 2500 50  0001 C CNN
+F 2 "Terminal_Blocks:TerminalBlock_Altech_AK300-2_P5.00mm" H 10050 2500 50  0001 C CNN
 F 3 "" H 10050 2500 50  0000 C CNN
-F 4 "ED2740-ND" H 10050 2500 60  0001 C CNN "digikey part no"
+F 4 "277-2518-ND" H 10050 2500 60  0001 C CNN "digikey part no"
 	1    10050 2500
 	0    1    1    0
@@
 F 0 "M5" H 10050 3610 50  0000 C CNN
 F 1 "E-MATCH" H 10050 3480 50  0000 C CNN
-F 2 "Terminal_Blocks:TerminalBlock_Pheonix_PT-3.5mm_2pol" H 10050 3550 50  0001 C CNN
+F 2 "Terminal_Blocks:TerminalBlock_Altech_AK300-2_P5.00mm" H 10050 3550 50  0001 C CNN
 F 3 "" H 10050 3550 50  0000 C CNN
-F 4 "ED2740-ND" H 10050 3550 60  0001 C CNN "digikey part no"
+F 4 "277-2518-ND" H 10050 3550 60  0001 C CNN "digikey part no"
 	1    10050 3550
 	0    1    1    0
@@
 F 0 "M6" H 10050 4510 50  0000 C CNN
 F 1 "E-MATCH" H 10050 4380 50  0000 C CNN
-F 2 "Terminal_Blocks:TerminalBlock_Pheonix_PT-3.5mm_2pol" H 10050 4450 50  0001 C CNN
+F 2 "Terminal_Blocks:TerminalBlock_Altech_AK300-2_P5.00mm" H 10050 4450 50  0001 C CNN
 F 3 "" H 10050 4450 50  0000 C CNN
-F 4 "ED2740-ND" H 10050 4450 60  0001 C CNN "digikey part no"
+F 4 "277-2518-ND" H 10050 4450 60  0001 C CNN "digikey part no"
 	1    10050 4450
 	0    1    1    0
@@
 F 0 "M7" H 10050 5560 50  0000 C CNN
 F 1 "E-MATCH" H 10050 5430 50  0000 C CNN
-F 2 "Terminal_Blocks:TerminalBlock_Pheonix_PT-3.5mm_2pol" H 10050 5500 50  0001 C CNN
+F 2 "Terminal_Blocks:TerminalBlock_Altech_AK300-2_P5.00mm" H 10050 5500 50  0001 C CNN
 F 3 "" H 10050 5500 50  0000 C CNN
-F 4 "ED2740-ND" H 10050 5500 60  0001 C CNN "digikey part no"
+F 4 "277-2518-ND" H 10050 5500 60  0001 C CNN "digikey part no"
 	1    10050 5500
 	0    1    1    0
@@
 12V
 $Comp
-L GND #PWR5
+L GND #PWR020
 U 1 1 56EC8173
 P 2700 5450
-F 0 "#PWR5" H 2700 5200 50  0001 C CNN
+F 0 "#PWR020" H 2700 5200 50  0001 C CNN
 F 1 "GND" H 2700 5300 50  0000 C CNN
 F 2 "" H 2700 5450 50  0000 C CNN
@@
 $EndComp
 $Comp
-L GND #PWR1
+L GND #PWR021
 U 1 1 56EFCFF7
 P 800 1800
-F 0 "#PWR1" H 800 1550 50  0001 C CNN
+F 0 "#PWR021" H 800 1550 50  0001 C CNN
 F 1 "GND" H 800 1650 50  0000 C CNN
 F 2 "" H 800 1800 50  0000 C CNN
@@
 $EndComp
 $Comp
-L GND #PWR3
+L GND #PWR022
 U 1 1 56EFD24E
 P 1300 2250
-F 0 "#PWR3" H 1300 2000 50  0001 C CNN
+F 0 "#PWR022" H 1300 2000 50  0001 C CNN
 F 1 "GND" H 1300 2100 50  0000 C CNN
 F 2 "" H 1300 2250 50  0000 C CNN
@@
 $EndComp
 $Comp
-L GND #PWR23
+L GND #PWR023
 U 1 1 56EFD3E4
 P 10400 2350
-F 0 "#PWR23" H 10400 2100 50  0001 C CNN
+F 0 "#PWR023" H 10400 2100 50  0001 C CNN
 F 1 "GND" H 10400 2200 50  0000 C CNN
 F 2 "" H 10400 2350 50  0000 C CNN
